File: PhotoSensor.brd (EAGLE design)
At the start: 38.1 x 17.8 mm, 7 parts, among them Q1 PT334-6B

Commit message: from Makefile
Parts:
- turned Q1 to 180 degrees
Connections:
- net GND: now also Q1.A; no longer Q1.K
- net OUT: now also Q1.K; no longer Q1.A
Other:
- board text added: "+"
- board text added: "-"
Changed lines of the file:
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@@
 <layer number="20" name="Dimension" color="15" fill="1" visible="yes" active="yes"/>
 <layer number="21" name="tPlace" color="7" fill="1" visible="yes" active="yes"/>
-<layer number="22" name="bPlace" color="7" fill="1" visible="yes" active="yes"/>
+<layer number="22" name="bPlace" color="14" fill="1" visible="yes" active="yes"/>
 <layer number="23" name="tOrigins" color="15" fill="1" visible="yes" active="yes"/>
-<layer number="24" name="bOrigins" color="15" fill="1" visible="yes" active="yes"/>
+<layer number="24" name="bOrigins" color="14" fill="1" visible="yes" active="yes"/>
 <layer number="25" name="tNames" color="7" fill="1" visible="yes" active="yes"/>
-<layer number="26" name="bNames" color="7" fill="1" visible="yes" active="yes"/>
+<layer number="26" name="bNames" color="6" fill="1" visible="yes" active="yes"/>
 <layer number="27" name="tValues" color="7" fill="1" visible="yes" active="yes"/>
-<layer number="28" name="bValues" color="7" fill="1" visible="yes" active="yes"/>
+<layer number="28" name="bValues" color="6" fill="1" visible="yes" active="yes"/>
 <layer number="29" name="tStop" color="7" fill="3" visible="no" active="yes"/>
 <layer number="30" name="bStop" color="7" fill="6" visible="no" active="yes"/>
@@
 <text x="25.4" y="11.43" size="0.8128" layer="22" rot="MR0" align="center">Cache Makers
 cachemakers.org</text>
+<text x="20.32" y="15.5575" size="1.27" layer="21" align="center">-</text>
+<text x="18.0975" y="12.3825" size="1.27" layer="21" align="center">+</text>
+<text x="27.94" y="15.5575" size="1.27" layer="21" align="center">-</text>
+<text x="25.7175" y="12.3825" size="1.27" layer="21" rot="R180" align="center">+</text>
+<text x="12.7" y="15.5575" size="1.27" layer="21" align="center">-</text>
+<text x="10.4775" y="12.3825" size="1.27" layer="21" align="center">+</text>
 </plain>
 <attributes>
@@
 </element>
 <element name="IR2" library="Optics" package="LED5MM" value="TSAL6100" x="11.43" y="13.97" smashed="yes">
-<attribute name="NAME" x="14.1859" y="13.97" size="1.27" layer="25" ratio="10" rot="R90" align="top-center"/>
+<attribute name="NAME" x="14.1859" y="12.7" size="1.27" layer="25" ratio="10" rot="R90" align="top-center"/>
 <attribute name="VALUE" x="11.4046" y="15.4559" size="0.8128" layer="28" ratio="10" rot="MR180" align="top-center"/>
 </element>
-<element name="Q1" library="Optics" package="LED5MM" value="PT334-6B" x="19.05" y="13.97" smashed="yes">
-<attribute name="NAME" x="21.8059" y="13.97" size="1.27" layer="25" ratio="10" rot="R90" align="top-center"/>
-<attribute name="VALUE" x="19.0246" y="15.7734" size="0.8128" layer="28" ratio="10" rot="MR180" align="top-center"/>
+<element name="Q1" library="Optics" package="LED5MM" value="PT334-6B" x="19.05" y="13.97" smashed="yes" rot="R180">
+<attribute name="NAME" x="16.2941" y="15.5575" size="1.27" layer="25" ratio="10" rot="R270" align="top-center"/>
+<attribute name="VALUE" x="19.0754" y="16.2941" size="0.8128" layer="28" ratio="10" rot="MR0" align="top-center"/>
 </element>
 <element name="2N3904" library="barbary_enterprises" package="TO-92-AMMO" value="2N3904" x="19.05" y="7.62" smashed="yes">
@@
 <signal name="GND">
 <contactref element="IR1" pad="K"/>
-<contactref element="Q1" pad="K"/>
+<contactref element="Q1" pad="A"/>
 <contactref element="JP1" pad="1"/>
 <wire x1="27.94" y1="13.97" x2="27.94" y2="13.335" width="0.8128" layer="16"/>
@@
 </signal>
 <signal name="OUT">
-<contactref element="Q1" pad="A"/>
+<contactref element="Q1" pad="K"/>
 <contactref element="R1" pad="P$1"/>
 <contactref element="JP1" pad="3"/>

Commit message: from Makefile
Parts:
- R1: value ? -> 10k
Changed lines of the file:
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@@
 <attribute name="VALUE" x="19.05" y="9.525" size="0.6096" layer="28" ratio="10" rot="MR0" align="top-center"/>
 </element>
-<element name="R1" library="barbary_enterprises" package="AXIAL-0.3" value="?" x="27.94" y="8.89" smashed="yes">
+<element name="R1" library="barbary_enterprises" package="AXIAL-0.3" value="10k" x="27.94" y="8.89" smashed="yes">
 <attribute name="NAME" x="25.7175" y="8.89" size="0.6096" layer="25" font="vector" align="center-left"/>
 <attribute name="VALUE" x="30.1625" y="8.89" size="0.8128" layer="21" font="vector" ratio="15" align="center-right"/>
