File: PhotoSensor.sch (EAGLE design)
At the start: 7 parts, among them Q1 PT334-6B

Commit message: updating readme.md
Other:
- note added: "User Hackable userhackable.com PhotoSensor"
Changed lines of the file:
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@@
 <sheet>
 <plain>
+<text x="35.56" y="48.26" size="1.778" layer="94">User Hackable
+userhackable.com
+PhotoSensor
+</text>
 </plain>
 <instances>
@@
 </schematic>
 </drawing>
+<compatibility>
+<note version="6.3" minversion="6.2.2" severity="warning">
+Since Version 6.2.2 text objects can contain more than one line,
+which will not be processed correctly with this version.
+</note>
+</compatibility>
 </eagle>

Commit message: from Makefile
Parts:
- R1: value ? -> 10k
Changed lines of the file:
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@@
 <part name="IR2" library="Optics" deviceset="LED" device="5MM" value="TSAL6100"/>
 <part name="2N3904" library="barbary_enterprises" deviceset="TRANSISTOR_NPN" device="TO-92-AMMO" value="2N3904"/>
-<part name="R1" library="barbary_enterprises" deviceset="RESISTOR" device="AXIAL-0.3" value="?"/>
+<part name="R1" library="barbary_enterprises" deviceset="RESISTOR" device="AXIAL-0.3" value="10k"/>
 <part name="R2" library="barbary_enterprises" deviceset="RESISTOR" device="AXIAL-0.3" value="33"/>
 <part name="SUPPLY1" library="barbary_enterprises" deviceset="5V" device=""/>
